File: IngestibleCapsule-Board_whole/processor.kicad_sch (KiCad schematic)
At the start: 21 parts, among them J1 TC2030-NL, J2 Conn_01x02_Pin, U1 STM32G473CCUx, Y1 ABM3, Y2 ABS07

Commit message: whole board
Parts:
- J2: footprint Connector_PinHeader_2.54mm:PinHeader_1x02_P2.54mm_Horizontal -> Connector_PinHeader_2.54mm:PinHeader_1x02_P2.54mm_Vertical
Connections:
- net GND: no longer U1.22 (PB10), U1.33 (PA11), U1.47 (PB9)
- no-connect marks 21 -> 24
Other:
- note removed: "FOR ROUTING PURPOSES"
Changed lines of the file:
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@@
 		)
 	)
-	(text "FOR ROUTING PURPOSES"
-		(exclude_from_sim no)
-		(at 234.696 83.058 0)
-		(effects
-			(font
-				(size 1.905 1.905)
-				(thickness 0.254)
-				(bold yes)
-			)
-		)
-	)
 	(junction
 		(at 55.88 167.64)
@@
 	)
 	(no_connect
+		(at 123.19 119.38)
+	)
+	(no_connect
 		(at 123.19 81.28)
 	)
@@
 	)
 	(no_connect
+		(at 123.19 121.92)
+	)
+	(no_connect
 		(at 123.19 127)
 	)
@@
 	)
 	(no_connect
+		(at 158.75 86.36)
+	)
+	(no_connect
 		(at 158.75 60.96)
 	)
@@
 	(wire
 		(pts
-			(xy 123.19 121.92) (xy 110.49 121.92)
-		)
-		(stroke
-			(width 0)
-			(type default)
-		)
-	)
-	(wire
-		(pts
 			(xy 29.21 123.19) (xy 29.21 121.92)
 		)
@@
 	(wire
 		(pts
-			(xy 158.75 86.36) (xy 171.45 86.36)
-		)
-		(stroke
-			(width 0)
-			(type default)
-		)
-	)
-	(wire
-		(pts
 			(xy 241.3 121.92) (xy 241.3 127)
 		)
@@
 	(wire
 		(pts
-			(xy 241.3 88.9) (xy 241.3 91.44)
-		)
-		(stroke
-			(width 0)
-			(type default)
-		)
-	)
-	(wire
-		(pts
 			(xy 135.89 48.26) (xy 135.89 50.8)
 		)
@@
 	(wire
 		(pts
-			(xy 123.19 119.38) (xy 110.49 119.38)
-		)
-		(stroke
-			(width 0)
-			(type default)
-		)
-	)
-	(wire
-		(pts
 			(xy 55.88 157.48) (xy 64.77 157.48)
 		)
@@
 	(wire
 		(pts
-			(xy 241.3 88.9) (xy 228.6 88.9)
-		)
-		(stroke
-			(width 0)
-			(type default)
-		)
-	)
-	(wire
-		(pts
 			(xy 123.19 88.9) (xy 104.14 88.9)
 		)
@@
 		)
 	)
-	(label "RT_GND"
-		(at 110.49 119.38 0)
-		(effects
-			(font
-				(size 1.27 1.27)
-			)
-			(justify left bottom)
-		)
-	)
-	(label "RT_GND"
-		(at 171.45 86.36 180)
-		(effects
-			(font
-				(size 1.27 1.27)
-			)
-			(justify right bottom)
-		)
-	)
 	(label "SWO"
 		(at 110.49 104.14 0)
@@
 		)
 	)
-	(label "RT_GND"
-		(at 228.6 88.9 0)
-		(effects
-			(font
-				(size 1.27 1.27)
-			)
-			(justify left bottom)
-		)
-	)
 	(label "SWCLK"
 		(at 57.15 50.8 180)
@@
 		)
 	)
-	(label "RT_GND"
-		(at 110.49 121.92 0)
-		(effects
-			(font
-				(size 1.27 1.27)
-			)
-			(justify left bottom)
-		)
-	)
 	(hierarchical_label "SPI_MISO"
 		(shape input)
@@
 	)
 	(symbol
-		(lib_id "power:GND")
-		(at 241.3 91.44 0)
-		(unit 1)
-		(exclude_from_sim no)
-		(in_bom yes)
-		(on_board yes)
-		(dnp no)
-		(fields_autoplaced yes)
-		(property "Reference" "#PWR018"
-			(at 241.3 97.79 0)
-			(effects
-				(font
-					(size 1.27 1.27)
-				)
-				(hide yes)
-			)
-		)
-		(property "Value" "GND"
-			(at 241.3 96.52 0)
-			(effects
-				(font
-					(size 1.27 1.27)
-				)
-			)
-		)
-		(property "Footprint" ""
-			(at 241.3 91.44 0)
-			(effects
-				(font
-					(size 1.27 1.27)
-				)
-				(hide yes)
-			)
-		)
-		(property "Datasheet" ""
-			(at 241.3 91.44 0)
-			(effects
-				(font
-					(size 1.27 1.27)
-				)
-				(hide yes)
-			)
-		)
-		(property "Description" "Power symbol creates a global label with name \"GND\" , ground"
-			(at 241.3 91.44 0)
-			(effects
-				(font
-					(size 1.27 1.27)
-				)
-				(hide yes)
-			)
-		)
-		(pin "1"
-		)
-		(instances
-			(project ""
-				(path "/c8668ce4-f244-4f6b-86d5-e45f0742e988/6af9e238-b56f-4881-bada-2247a4bc5709"
-					(reference "#PWR018")
-					(unit 1)
-				)
-			)
-		)
-	)
-	(symbol
 		(lib_id "Device:C_Small")
 		(at 64.77 162.56 0)
@@
 			)
 		)
-		(property "Footprint" "Connector_PinHeader_2.54mm:PinHeader_1x02_P2.54mm_Horizontal"
+		(property "Footprint" "Connector_PinHeader_2.54mm:PinHeader_1x02_P2.54mm_Vertical"
 			(at 83.82 163.83 0)
 			(effects
