File: IngestibleCapsule-Board_whole/IngestibleCapsule-Board_whole.kicad_pcb (KiCad board)
At the start: 2 copper layers, 48 parts, among them J1 TC2030-NL, J2 Conn_01x02_Pin, U1 STM32G473CCUx, U2 MLX90640, U3 ADXL343, U4 W25Q16JVSS, U5 SR1010, Y1 ABM3, Y2 ABS07, Y3 ABS07

Commit message: whole board
Parts:
- J2: footprint Connector_PinHeader_2.54mm:PinHeader_1x02_P2.54mm_Horizontal -> Connector_PinHeader_2.54mm:PinHeader_1x02_P2.54mm_Vertical
- moved U4 97.4 mm to (58.8, 84.4)
- moved R8 95.8 mm to (55.1, 80.5), turned to 180 degrees
- moved C14 91.3 mm to (62.6, 80.5)
- moved C12 84.7 mm to (55.1, 88.4)
- moved U3 82.7 mm to (65.2, 96.8), turned to 90 degrees
- moved U2 78.7 mm to (58.4, 94.5), turned to 180 degrees
- moved C13 75.4 mm to (63.4, 99.7)
- moved R7 73.1 mm to (64.0, 91.8), turned to -90 degrees
- moved R6 63.9 mm to (72.4, 95.8), turned to 180 degrees
- moved R5 63.8 mm to (72.4, 94.5), turned to 180 degrees
- moved Y1 61.3 mm to (74.5, 80.3), turned to 180 degrees
- moved R9 58.6 mm to (65.7, 78.1)
- moved R1 58.4 mm to (70.2, 81.7), turned to 180 degrees
- moved R3 56.7 mm to (72.4, 83.0)
- moved R10 52.5 mm to (71.7, 76.7), turned to 180 degrees
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Connections:
- U1 pad 22: GND -> unconnected-(U1-PB10-Pad22)
- U1 pad 33: GND -> unconnected-(U1-PA11-Pad33)
- U1 pad 47: GND -> unconnected-(U1-PB9-Pad47)
Routing:
- net GND: track 0.00 -> 50.5 mm, vias 0 -> 88
- net +3.3V: track 0.00 -> 30.1 mm, vias 0 -> 4
- net /Memory/MEM_MISO: track 0.00 -> 24.7 mm, vias 0 -> 2
- net /Processor/I2C_SDA: track 0.00 -> 19.2 mm, vias 0 -> 2
- net /Memory/MEM_MOSI: track 0.00 -> 18.7 mm
- net /Processor/I2C_SCL: track 0.00 -> 18.4 mm, vias 0 -> 2
- net /Processor/NRST: track 0.00 -> 17.8 mm, vias 0 -> 2
- net /Memory/MEM_SCK: track 0.00 -> 17.8 mm, vias 0 -> 3
- net /Memory/MEM_CS_IN: track 0.00 -> 17.3 mm
- net /Processor/RF_IRQ_IN: track 0.00 -> 11.8 mm, vias 0 -> 2
- net /Processor/RF_CS_OUT: track 0.00 -> 11.6 mm, vias 0 -> 2
- net Net-(U1-PF0): track 0.00 -> 8.45 mm
- net Net-(U5-XTAL_C2): track 0.00 -> 8.05 mm
- net Net-(U1-PC14): track 0.00 -> 7.15 mm
- net Net-(U1-PC15): track 0.00 -> 7.11 mm
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- added copper zone on F.Cu, net +3.3V
- added copper zone on B.Cu, net GND
- added copper zone on F.Cu, net GND
Other:
- board outline added: 37.4 x 54.2 mm
