File: IngestibleCapsule-Board_v2/memory.kicad_sch (KiCad schematic)
At the start: 3 parts, among them U4 W25Q16JVSS

Commit message: full v2 implementation, has 5 circles connected by mousebites
Parts:
- renumbered C14 to C15
Changed lines of the file:
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@@
 		(dnp no)
 		(fields_autoplaced yes)
-		(property "Reference" "#PWR072"
+		(property "Reference" "#PWR052"
 			(at 129.54 97.79 0)
 			(effects
@@
 			(project "IngestibleCapsule-Board"
 				(path "/c8668ce4-f244-4f6b-86d5-e45f0742e988/664eb997-5495-46fb-a0f6-a32895b81cf6"
-					(reference "#PWR072")
+					(reference "#PWR052")
 					(unit 1)
 				)
@@
 		(dnp no)
 		(fields_autoplaced yes)
-		(property "Reference" "#PWR073"
+		(property "Reference" "#PWR050"
 			(at 96.52 107.95 0)
 			(effects
@@
 			(project "IngestibleCapsule-Board"
 				(path "/c8668ce4-f244-4f6b-86d5-e45f0742e988/664eb997-5495-46fb-a0f6-a32895b81cf6"
-					(reference "#PWR073")
+					(reference "#PWR050")
 					(unit 1)
 				)
@@
 		(dnp no)
 		(fields_autoplaced yes)
-		(property "Reference" "#PWR070"
+		(property "Reference" "#PWR048"
 			(at 76.2 114.3 0)
 			(effects
@@
 			(project "IngestibleCapsule-Board"
 				(path "/c8668ce4-f244-4f6b-86d5-e45f0742e988/664eb997-5495-46fb-a0f6-a32895b81cf6"
-					(reference "#PWR070")
+					(reference "#PWR048")
 					(unit 1)
 				)
@@
 		(dnp no)
 		(fields_autoplaced yes)
-		(property "Reference" "C14"
+		(property "Reference" "C15"
 			(at 132.08 85.0962 0)
 			(effects
@@
 			(project "IngestibleCapsule-Board"
 				(path "/c8668ce4-f244-4f6b-86d5-e45f0742e988/664eb997-5495-46fb-a0f6-a32895b81cf6"
-					(reference "C14")
+					(reference "C15")
 					(unit 1)
 				)
@@
 		(dnp no)
 		(fields_autoplaced yes)
-		(property "Reference" "#PWR068"
+		(property "Reference" "#PWR049"
 			(at 96.52 72.39 0)
 			(effects
@@
 			(project "IngestibleCapsule-Board"
 				(path "/c8668ce4-f244-4f6b-86d5-e45f0742e988/664eb997-5495-46fb-a0f6-a32895b81cf6"
-					(reference "#PWR068")
+					(reference "#PWR049")
 					(unit 1)
 				)
@@
 		(dnp no)
 		(fields_autoplaced yes)
-		(property "Reference" "#PWR069"
+		(property "Reference" "#PWR047"
 			(at 67.31 72.39 0)
 			(effects
@@
 			(project "IngestibleCapsule-Board"
 				(path "/c8668ce4-f244-4f6b-86d5-e45f0742e988/664eb997-5495-46fb-a0f6-a32895b81cf6"
-					(reference "#PWR069")
+					(reference "#PWR047")
 					(unit 1)
 				)
@@
 		(dnp no)
 		(fields_autoplaced yes)
-		(property "Reference" "#PWR071"
+		(property "Reference" "#PWR051"
 			(at 129.54 85.09 0)
 			(effects
@@
 			(project "IngestibleCapsule-Board"
 				(path "/c8668ce4-f244-4f6b-86d5-e45f0742e988/664eb997-5495-46fb-a0f6-a32895b81cf6"
-					(reference "#PWR071")
-					(unit 1)
-				)
+					(reference "#PWR051")
+					(unit 1)
+				)
