File: IngestibleCapsule-Board_v2/processor.kicad_sch (KiCad schematic)
At the start: 21 parts, among them J1 TC2030-NL, U1 STM32G473CCUx, Y1 ABM3, Y2 ABS07

Commit message: full v2 implementation, has 5 circles connected by mousebites
Parts:
- renumbered C5 to C1, C2 to C10, C3 to C11, C4 to C12, C11 to C2, C6 to C3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
